File: RideHeightSensor/RideHeightSensor.kicad_sch (KiCad schematic)
At the start: 8 parts

Commit message: Add PicoCANCode base
Parts:
- added J?: CONN_01x02, footprints:PinHeader_1x02_P2.54mm_Vertical, symbol baja_schematics:CONN_01x02
- added J?: INPUT, symbol Connector:Screw_Terminal_01x02
Connections:
- net at R?.1, U?.1: no longer J?.2 (Pin_2), U?.3 (+)
- new net: J?.2 (Pin_2), U?.3 (+)
- new net CANH: J?.2 (Pin_2), J?.2 (Pin_2)
- new net CANL: J?.1 (Pin_1), J?.1 (Pin_1)
Other:
- note added: "MUST ADD BOARD ID"
Changed lines of the file:
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@@
 (kicad_sch (version 20211123) (generator eeschema)
   (paper "A4")
-  (junction (at 64.77 35.56) (diameter 0) (color 0 0 0 0)
-  )
-  (junction (at 81.28 38.1) (diameter 0) (color 0 0 0 0)
-  )
   (junction (at 81.28 45.72) (diameter 0) (color 0 0 0 0)
   )
@@
     (stroke (width 0) (type default) (color 0 0 0 0))
   )
-  (wire (pts (xy 81.28 38.1) (xy 81.28 31.75))
-    (stroke (width 0) (type default) (color 0 0 0 0))
-  )
   (wire (pts (xy 137.922 22.86) (xy 142.24 22.86))
     (stroke (width 0) (type default) (color 0 0 0 0))
@@
     (stroke (width 0) (type default) (color 0 0 0 0))
   )
-  (wire (pts (xy 45.72 35.56) (xy 64.77 35.56))
-    (stroke (width 0) (type default) (color 0 0 0 0))
-  )
-  (wire (pts (xy 64.77 31.75) (xy 64.77 35.56))
+  (wire (pts (xy 45.72 35.56) (xy 66.04 35.56))
     (stroke (width 0) (type default) (color 0 0 0 0))
   )
@@
     (stroke (width 0) (type default) (color 0 0 0 0))
   )
-  (wire (pts (xy 81.28 31.75) (xy 64.77 31.75))
+  (wire (pts (xy 155.956 52.578) (xy 163.068 52.578))
     (stroke (width 0) (type default) (color 0 0 0 0))
   )
@@
     (stroke (width 0) (type default) (color 0 0 0 0))
   )
+  (wire (pts (xy 155.956 50.038) (xy 163.068 50.038))
+    (stroke (width 0) (type default) (color 0 0 0 0))
+  )
   (wire (pts (xy 127 35.56) (xy 145.288 35.56))
     (stroke (width 0) (type default) (color 0 0 0 0))
   )
-  (wire (pts (xy 64.77 35.56) (xy 66.04 35.56))
-    (stroke (width 0) (type default) (color 0 0 0 0))
-  )
   (wire (pts (xy 81.28 45.72) (xy 91.44 45.72))
     (stroke (width 0) (type default) (color 0 0 0 0))
@@
   (wire (pts (xy 142.24 22.86) (xy 142.24 25.4))
     (stroke (width 0) (type default) (color 0 0 0 0))
+  )
+  (text "MUST ADD BOARD ID" (at 114.3 80.264 0)
+    (effects (font (size 5 5)) (justify left bottom))
+  )
+  (label "CANH" (at 155.956 52.578 0)
+    (effects (font (size 1.27 1.27)) (justify left bottom))
+  )
+  (label "CANH" (at 44.704 75.692 0)
+    (effects (font (size 1.27 1.27)) (justify left bottom))
+  )
+  (label "CANL" (at 44.704 73.152 0)
+    (effects (font (size 1.27 1.27)) (justify left bottom))
+  )
+  (label "CANL" (at 155.956 50.038 0)
+    (effects (font (size 1.27 1.27)) (justify left bottom))
   )
   (symbol (lib_id "Amplifier_Operational:LMC6484") (at 73.66 38.1 0) (unit 1)
@@
     (pin "1")
   )
+  (symbol (lib_id "baja_schematics:CONN_01x02") (at 168.148 50.038 0) (unit 1)
+    (in_bom yes) (on_board yes) (fields_autoplaced)
+    (property "Reference" "J?" (id 0) (at 170.18 50.0379 0)
+      (effects (font (size 1.27 1.27)) (justify left))
+    )
+    (property "Value" "CONN_01x02" (id 1) (at 170.18 52.5779 0)
+      (effects (font (size 1.27 1.27)) (justify left))
+    )
+    (property "Footprint" "footprints:PinHeader_1x02_P2.54mm_Vertical" (id 2) (at 165.608 50.038 0)
+      (effects (font (size 1.27 1.27)) hide)
+    )
+    (property "Datasheet" "https://katalog.we-online.de/em/datasheet/6130xx11121.pdf" (id 3) (at 168.148 47.498 0)
+      (effects (font (size 1.27 1.27)) hide)
+    )
+    (property "MFN" "DK" (id 4) (at 170.688 44.958 0)
+      (effects (font (size 1.27 1.27)) hide)
+    )
+    (property "MPN" "732-5315-ND" (id 5) (at 173.228 42.418 0)
+      (effects (font (size 1.27 1.27)) hide)
+    )
+    (pin "1")
+    (pin "2")
+  )
   (symbol (lib_id "power:GND") (at 81.28 53.34 0) (unit 1)
     (in_bom yes) (on_board yes)
@@
     )
     (property "Datasheet" "~" (id 3) (at 81.28 49.53 0)
+      (effects (font (size 1.27 1.27)) hide)
+    )
+    (pin "1")
+    (pin "2")
+  )
+  (symbol (lib_id "Connector:Screw_Terminal_01x02") (at 39.624 73.152 0) (mirror y) (unit 1)
+    (in_bom yes) (on_board yes) (fields_autoplaced)
+    (property "Reference" "J?" (id 0) (at 39.624 67.056 0))
+    (property "Value" "INPUT" (id 1) (at 39.624 69.596 0))
+    (property "Footprint" "" (id 2) (at 39.624 73.152 0)
+      (effects (font (size 1.27 1.27)) hide)
+    )
+    (property "Datasheet" "~" (id 3) (at 39.624 73.152 0)
       (effects (font (size 1.27 1.27)) hide)
     )
@@
       (reference "J?") (unit 1) (value "Conn_01x07") (footprint "Connector_PinHeader_2.54mm:PinHeader_1x07_P2.54mm_Vertical")
     )
+    (path "/1ce44af8-cce8-4ca9-94c3-991d409c5a51"
+      (reference "J?") (unit 1) (value "CONN_01x02") (footprint "footprints:PinHeader_1x02_P2.54mm_Vertical")
+    )
     (path "/22575fc9-293b-4049-9f8d-8c4f45e59821"
       (reference "J?") (unit 1) (value "Ride_Height_Sensor") (footprint "")
     )
+    (path "/69a272ff-5214-4d38-8ac1-8acff7aadf6f"
+      (reference "J?") (unit 1) (value "INPUT") (footprint "")
+    )
     (path "/914af70e-27b2-4a76-ba47-2d4794c83cc9"

Commit message: Update RHS schematic
Connections:
- net GND: no longer U?.2 (-)
- net at R?.1, U?.1: now also U?.2 (-)
Other:
- moved on the sheet: U?A
Changed lines of the file:
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@@
   (junction (at 81.28 45.72) (diameter 0) (color 0 0 0 0)
   )
+  (junction (at 77.216 38.1) (diameter 0) (color 0 0 0 0)
+  )
   (wire (pts (xy 142.24 25.4) (xy 145.288 25.4))
     (stroke (width 0) (type default) (color 0 0 0 0))
@@
     (stroke (width 0) (type default) (color 0 0 0 0))
   )
-  (wire (pts (xy 45.72 35.56) (xy 66.04 35.56))
+  (wire (pts (xy 77.216 38.1) (xy 81.28 38.1))
+    (stroke (width 0) (type default) (color 0 0 0 0))
+  )
+  (wire (pts (xy 45.72 35.56) (xy 60.198 35.56))
     (stroke (width 0) (type default) (color 0 0 0 0))
   )
@@
     (stroke (width 0) (type default) (color 0 0 0 0))
   )
+  (wire (pts (xy 60.198 40.64) (xy 60.198 45.466))
+    (stroke (width 0) (type default) (color 0 0 0 0))
+  )
+  (wire (pts (xy 77.216 45.466) (xy 77.216 38.1))
+    (stroke (width 0) (type default) (color 0 0 0 0))
+  )
   (wire (pts (xy 127 35.56) (xy 145.288 35.56))
     (stroke (width 0) (type default) (color 0 0 0 0))
   )
+  (wire (pts (xy 60.198 45.466) (xy 77.216 45.466))
+    (stroke (width 0) (type default) (color 0 0 0 0))
+  )
   (wire (pts (xy 81.28 45.72) (xy 91.44 45.72))
     (stroke (width 0) (type default) (color 0 0 0 0))
@@
   )
   (wire (pts (xy 142.24 22.86) (xy 142.24 25.4))
+    (stroke (width 0) (type default) (color 0 0 0 0))
+  )
+  (wire (pts (xy 75.438 38.1) (xy 77.216 38.1))
     (stroke (width 0) (type default) (color 0 0 0 0))
   )
@@
     (effects (font (size 1.27 1.27)) (justify left bottom))
   )
-  (symbol (lib_id "Amplifier_Operational:LMC6484") (at 73.66 38.1 0) (unit 1)
-    (in_bom yes) (on_board yes) (fields_autoplaced)
-    (property "Reference" "U?" (id 0) (at 73.66 27.94 0))
-    (property "Value" "LMC6484" (id 1) (at 73.66 30.48 0))
-    (property "Footprint" "" (id 2) (at 72.39 35.56 0)
-      (effects (font (size 1.27 1.27)) hide)
-    )
-    (property "Datasheet" "http://www.ti.com/lit/ds/symlink/lmc6484.pdf" (id 3) (at 74.93 33.02 0)
+  (symbol (lib_id "Amplifier_Operational:LMC6484") (at 67.818 38.1 0) (unit 1)
+    (in_bom yes) (on_board yes) (fields_autoplaced)
+    (property "Reference" "U?" (id 0) (at 67.818 27.94 0))
+    (property "Value" "LMC6484" (id 1) (at 67.818 30.48 0))
+    (property "Footprint" "" (id 2) (at 66.548 35.56 0)
+      (effects (font (size 1.27 1.27)) hide)
+    )
+    (property "Datasheet" "http://www.ti.com/lit/ds/symlink/lmc6484.pdf" (id 3) (at 69.088 33.02 0)
       (effects (font (size 1.27 1.27)) hide)
     )
@@
     (pin "1")
   )
-  (symbol (lib_id "power:GND") (at 66.04 40.64 0) (unit 1)
-    (in_bom yes) (on_board yes) (fields_autoplaced)
-    (property "Reference" "#PWR?" (id 0) (at 66.04 46.99 0)
-      (effects (font (size 1.27 1.27)) hide)
-    )
-    (property "Value" "GND" (id 1) (at 66.04 45.72 0))
-    (property "Footprint" "" (id 2) (at 66.04 40.64 0)
-      (effects (font (size 1.27 1.27)) hide)
-    )
-    (property "Datasheet" "" (id 3) (at 66.04 40.64 0)
-      (effects (font (size 1.27 1.27)) hide)
-    )
-    (pin "1")
-  )
   (sheet_instances
     (path "/" (page "1"))
@@
       (reference "#PWR?") (unit 1) (value "GND") (footprint "")
     )
-    (path "/f7362adc-fdbc-4ae0-8036-18646e25ead4"
-      (reference "#PWR?") (unit 1) (value "GND") (footprint "")
-    )
